Commit message: Adds config, updates newrobot files
newrobot.xacro now includes real laser meshes, and newrobot.urdf is now the result of converting robot.xacro to urdf

File: urdf/newrobot.xacro (robot description, xacro)
@@ -1,135 +1,116 @@
-<?xml version="1.0" ?>
-<!-- =================================================================================== -->
-<!-- |    This document was autogenerated by xacro from urdf/robot.xacro               | -->
-<!-- |    EDITING THIS FILE BY HAND IS NOT RECOMMENDED                                 | -->
-<!-- =================================================================================== -->
+<?xml version="1.0"?>
 <robot name="robot1" xmlns:xacro="http://www.ros.org/wiki/xacro">
-  <link name="base">
-    <visual>
-      <origin xyz="0 0 0.99"/>
-      <geometry>
-        <box size="0.94 0.78 1.98"/>
-      </geometry>
-    </visual>
-    <collision>
-      <geometry>
-        <box size="0.94 0.78 1.98"/>
-      </geometry>
-    </collision>
-  </link>
-  <link name="laser_vert_bottom">
-    <visual>
-      <origin rpy="3.1355 -1.3045 0.0025" xyz="0.3158 -0.0021 0.5100"/>
-      <geometry>
-        <box size="0.062 0.062 0.087"/>
-      </geometry>
-    </visual>
-  </link>
-  <link name="laser_vert_top_right">
-    <visual>
-      <origin rpy="-1.1760 0.6313 -1.9377" xyz="0.2978 -0.1450 1.8451"/>
-      <geometry>
-        <box size="0.062 0.062 0.087"/>
-      </geometry>
-    </visual>
-  </link>
-  <link name="laser_vert_top_left">
-    <visual>
-      <origin rpy="1.1780 0.6198 1.9560" xyz="0.2997 0.1531 1.8443"/>
-      <geometry>
-        <box size="0.062 0.062 0.087"/>
-      </geometry>
-    </visual>
-  </link>
-  <link name="laser_horiz">
-    <visual>
-      <origin rpy="-0.0012 0.1146 -0.0015" xyz="0.2325 0.0001 1.9201"/>
-      <geometry>
-        <cylinder length="0.072" radius="0.052"/>
-      </geometry>
-    </visual>
-    <collision>
-      <origin rpy="-0.0012 0.1146 -0.0015" xyz="0.2325 0.0001 1.9201"/>
-      <geometry>
-        <cylinder length="0.072" radius="0.052"/>
-      </geometry>
-    </collision>
-  </link>
-  <joint name="base_laser_vert_bottom_joint" type="fixed">
-    <parent link="base"/>
-    <child link="laser_vert_bottom"/>
-    <origin xyz="0.3158 -0.0021 0.5100"/>
-  </joint>
-  <joint name="base_laser_vert_top_right_joint" type="fixed">
-    <parent link="base"/>
-    <child link="laser_vert_top_right"/>
-    <origin xyz="0.2978 -0.1450 1.8451"/>
-  </joint>
-  <joint name="base_laser_vert_top_left_joint" type="fixed">
-    <parent link="base"/>
-    <child link="laser_vert_top_left"/>
-    <origin xyz="0.2997 0.1531 1.8443"/>
-  </joint>
-  <joint name="base_laser_horiz_joint" type="fixed">
-    <parent link="base"/>
-    <child link="laser_horiz"/>
-    <origin xyz="0.2325 0.001 1.9201"/>
-  </joint>
-  <link name="wheel_left">
-    <visual>
-      <origin rpy="-1.5707 0 0" xyz="-0.1 0.4 0"/>
-      <geometry>
-        <cylinder length="0.05" radius="0.2"/>
-      </geometry>
-    </visual>
-    <collision>
-      <origin rpy="-1.5707 0 0" xyz="-0.1 0.4 0"/>
-      <geometry>
-        <cylinder length="0.05" radius="0.2"/>
-      </geometry>
-    </collision>
-  </link>
-  <joint name="base_wheel_left_joint" type="fixed">
-    <parent link="base"/>
-    <child link="wheel_left"/>
-    <origin xyz="-0.1 0.4 0"/>
-  </joint>
-  <link name="wheel_right">
-    <visual>
-      <origin rpy="-1.5707 0 0" xyz="-0.1 -0.4 0"/>
-      <geometry>
-        <cylinder length="0.05" radius="0.2"/>
-      </geometry>
-    </visual>
-    <collision>
-      <origin rpy="-1.5707 0 0" xyz="-0.1 -0.4 0"/>
-      <geometry>
-        <cylinder length="0.05" radius="0.2"/>
-      </geometry>
-    </collision>
-  </link>
-  <joint name="base_wheel_right_joint" type="fixed">
-    <parent link="base"/>
-    <child link="wheel_right"/>
-    <origin xyz="-0.1 0.4 0"/>
-  </joint>
-  <link name="wheel_center">
-    <visual>
-      <origin rpy="-1.5707 0 0" xyz="-0.1 0.0 0"/>
-      <geometry>
-        <cylinder length="0.05" radius="0.2"/>
-      </geometry>
-    </visual>
-    <collision>
-      <origin rpy="-1.5707 0 0" xyz="-0.1 0.0 0"/>
-      <geometry>
-        <cylinder length="0.05" radius="0.2"/>
-      </geometry>
-    </collision>
-  </link>
-  <joint name="base_wheel_center_joint" type="fixed">
-    <parent link="base"/>
-    <child link="wheel_center"/>
-    <origin xyz="-0.1 0.4 0"/>
-  </joint>
+	<xacro:include filename="$(find gazebo_plugins)/test/multi_robot_scenario/xacro/laser/hokuyo.xacro" />
+	<xacro:include filename="$(find velodyne_description)/urdf/VLP-16.urdf.xacro"/>
+	<link name="base">
+		<visual>
+			<origin xyz = "0 0 0.99"/>
+			<geometry>
+				<box size="0.94 0.78 1.98"/>
+			</geometry>
+		</visual>
+		<collision>
+			<geometry>
+				<box size="0.94 0.78 1.98"/>
+			</geometry>
+		</collision>
+	</link>
+	<xacro:laser name="laser_vert_bottom" parent="base" xyz="0.3157894464801903
+-0.002068548615034871 0.5099999434059285" rpy="3.1354753 -1.3045001 0.0024658"
+meshes="package://gazebo_plugins/test/multi_robot_scenario/meshes/laser" />
+<!--
+	<link name="laser_vert_bottom">
+		<visual>
+			<origin xyz="0.3158 -0.0021 0.5100" rpy="3.1355 -1.3045 0.0025"/>
+			<geometry>
+				<box size="0.062 0.062 0.087"/>
+			</geometry>
+		</visual>
+	</link> -->
+	<xacro:laser name="laser_vert_top_right" parent="base" xyz="0.2978 -0.1450 1.8451" rpy="-1.1760 0.6313 -1.9377" meshes="package://gazebo_plugins/test/multi_robot_scenario/meshes/laser" />
+	<!--
+	<link name="laser_vert_top_right">
+		<visual>
+			<origin xyz = "0.2978 -0.1450 1.8451" rpy = "-1.1760 0.6313 -1.9377"/>
+			<geometry>
+				<box size="0.062 0.062 0.087"/>
+			</geometry>
+		</visual>
+	</link>
+-->
+	<xacro:laser name="laser_vert_top_left" parent="base" xyz="0.2997 0.1531 1.8443" rpy="1.1780 0.6198 1.9560" meshes="package://gazebo_plugins/test/multi_robot_scenario/meshes/laser" />
+<!--
+	<link name="laser_vert_top_left">
+		<visual>
+			<origin xyz = "0.2997 0.1531 1.8443" rpy = "1.1780 0.6198 1.9560"/>
+			<geometry>
+				<box size = "0.062 0.062 0.087"/>
+			</geometry>
+		</visual>
+	</link>
+-->
+	<VLP-16 parent="base" name="laser_horiz" topic="laser_horiz/packets" hz="10" samples="440" gpu="false">
+		<origin xyz="0.2325416305773505 -0.0001380069427607134 1.920122926231907" rpy="-0.0012068 0.114646 -0.0015308" />
+	</VLP-16>
+<!--
+	<link name="laser_horiz">
+		<visual>
+			<origin xyz = "0.2325 0.0001 1.9201" rpy = "-0.0012 0.1146 -0.0015"/>
+			<geometry>
+				<cylinder radius = "0.052" length = "0.072"/>
+			</geometry>
+		</visual>
+		<collision>
+			<origin xyz = "0.2325 0.0001 1.9201" rpy = "-0.0012 0.1146 -0.0015"/>
+			<geometry>
+				<cylinder radius = "0.052" length = "0.072"/>
+			</geometry>
+		</collision>
+	</link>
+-->
+	<joint name="base_laser_vert_bottom_joint" type="fixed">
+		<parent link="base"/>
+		<child link="laser_vert_bottom"/>
+		<origin xyz="0.3158 -0.0021 0.5100"/>
+	</joint>
+	<joint name="base_laser_vert_top_right_joint" type="fixed">
+		<parent link="base"/>
+		<child link="laser_vert_top_right"/>
+		<origin xyz="0.2978 -0.1450 1.8451"/>
+	</joint>
+	<joint name="base_laser_vert_top_left_joint" type="fixed">
+		<parent link="base"/>
+		<child link="laser_vert_top_left"/>
+		<origin xyz="0.2997 0.1531 1.8443"/>
+	</joint>
+	<joint name="base_laser_horiz_joint" type="fixed">
+		<parent link="base"/>
+		<child link="laser_horiz"/>
+		<origin xyz="0.2325 0.001 1.9201"/>
+	</joint>
+	<xacro:macro name="xacro_name" params="suffix reflect shift size">
+		<link name="wheel_${suffix}">
+			<visual>
+				<origin xyz="${shift} ${reflect * 0.4} 0" rpy="-1.5707 0 0"/>
+				<geometry>
+					<cylinder radius="${0.2+size}" length="0.05"/>
+				</geometry>
+			</visual>
+			<collision>
+				<origin xyz="${shift} ${0.4*reflect} 0" rpy="-1.5707 0 0"/>
+				<geometry>
+					<cylinder radius="${0.2+size}" length="0.05"/>
+				</geometry>
+			</collision>
+		</link>
+		<joint name="base_wheel_${suffix}_joint" type="continuous">
+			<parent link="base"/>
+			<child link="wheel_${suffix}"/>
+			<origin xyz="${shift} ${reflect * 0.4} 0"/>
+			<axis xyz="0 1 0"/>
+		</joint>
+	</xacro:macro>
+	<xacro:xacro_name suffix="left" reflect="1" shift="-0.1" size="0"/>
+	<xacro:xacro_name suffix="right" reflect="-1" shift="-0.1" size="0"/>
+	<xacro:xacro_name suffix="center" reflect="0" shift="0.1" size="-0.05"/>
 </robot>
